Commit message: fix lidar error

File: install/sese/share/sese/description/lidar.xacro (robot description, xacro)
@@ -29,5 +29,5 @@
             <update_rate>5</update_rate>
             <ray>
-            <!-- <scan>
+            <scan>
                 <horizontal>
                 <samples>360</samples>
@@ -36,6 +36,6 @@
                 <max_angle>6.280000</max_angle>
                 </horizontal>
-            </scan> -->
-            <scan>
+            </scan>
+            <!-- <scan>
                 <horizontal>
                 <samples>180</samples>
@@ -44,5 +44,5 @@
                 <max_angle>-1.570000</max_angle>
                 </horizontal>
-            </scan>
+            </scan> -->
             <range>
                 <min>0.50000</min>
@@ -56,7 +56,7 @@
             </noise>
             </ray>
-            <plugin name="my_scan" filename="libgazebo_ros_ray_sensor.so">
+            <plugin name="scan" filename="libgazebo_ros_ray_sensor.so">
             <ros>
-                <remapping>~/out:=my_scan</remapping>
+                <remapping>~/out:=scan</remapping>
             </ros>
             <output_type>sensor_msgs/LaserScan</output_type>

File: install/sese/share/sese/description/robot_core.xacro (robot description, xacro)
@@ -133,5 +133,5 @@
         <mu2 value="0.001"/>
     </gazebo>
-    <!-- <link name="imu_link">
+    <link name="imu_link">
         <visual>
             <geometry>
@@ -148,14 +148,14 @@
             <origin xyz="0 0 0" rpy="0 0 0"/>
         </xacro:inertial_box>
-    </link> -->
-    <!-- <gazebo reference="imu_link">
+    </link>
+    <gazebo reference="imu_link">
         <material>Gazebo/Red</material>
-    </gazebo> -->
-    <!-- <joint name="imu_joint" type="fixed">
+    </gazebo>
+    <joint name="imu_joint" type="fixed">
     <parent link="base_link"/>
     <child link="imu_link"/>
     <origin xyz="0 0 0.15"/>
-    </joint> -->
-    <!-- <gazebo reference="imu_link">
+    </joint>
+    <gazebo reference="imu_link">
     <sensor name="imu_sensor" type="imu">
     <plugin filename="libgazebo_ros_imu_sensor.so" name="imu_plugin">
@@ -224,4 +224,4 @@
         </imu>
     </sensor>
-    </gazebo> -->
+    </gazebo>
 </robot>
